Commit message: Correction typo "rigth" sur le nom de "arm_pitch"

File: Data/sigmaban.urdf (robot description, URDF)
Before this commit: robot URDF, 26 links, 25 joints
Joints:
- removed joint rigth_arm_pitch
- added joint right_arm_pitch: type continuous, parent trunk_link, child right_arm_pitch_link, origin xyz=0.0111273159824815 -0.0463847022119884 0.141000000000006 rpy=4.91888973129517E-16 6.34190653024847E-17 -0.00107822069516516, axis 0 1 0
