Commit message: GrosbanToe model: adding arms

File: Data/GrosbanToe.urdf (robot description, URDF)
Before this commit: robot DummyRobot, 15 links, 14 joints
Links:
- added link left_elbow_link, mass 1.0
- added link left_hand_link, mass 1.0
- added link left_shoulder_pitch_link, mass 1.0
- added link left_shoulder_roll_link, mass 1.0
- added link right_elbow_link, mass 1.0
- added link right_hand_link, mass 1.0
- added link right_shoulder_pitch_link, mass 1.0
- added link right_shoulder_roll_link, mass 1.0
Joints:
- added joint left_elbow: type continuous, parent left_shoulder_roll_link, child left_elbow_link, origin xyz=0 0 -0.1 rpy=0 0 0, axis 0 1 0
- added joint left_hand: type fixed, parent left_elbow_link, child left_hand_link, origin xyz=0 0 -0.1 rpy=0 0 0
- added joint left_shoulder_pitch: type continuous, parent trunk_link, child left_shoulder_pitch_link, origin xyz=0 0.15 0.1 rpy=0 0 0, axis 0 1 0
- added joint left_shoulder_roll: type continuous, parent left_shoulder_pitch_link, child left_shoulder_roll_link, origin xyz=0 0 0 rpy=0 0 0, axis 1 0 0
- added joint right_elbow: type continuous, parent right_shoulder_roll_link, child right_elbow_link, origin xyz=0 0 -0.1 rpy=0 0 0, axis 0 1 0
- added joint right_hand: type fixed, parent right_elbow_link, child right_hand_link, origin xyz=0 0 -0.1 rpy=0 0 0
- added joint right_shoulder_pitch: type continuous, parent trunk_link, child right_shoulder_pitch_link, origin xyz=0 -0.15 0.1 rpy=0 0 0, axis 0 1 0
- added joint right_shoulder_roll: type continuous, parent right_shoulder_pitch_link, child right_shoulder_roll_link, origin xyz=0 0 0 rpy=0 0 0, axis 1 0 0

Commit message: Adding head and tips for foot

File: Data/GrosbanToe.urdf (robot description, URDF)
Before this commit: robot DummyRobot, 23 links, 22 joints
Links:
- added link head_pitch_link, mass 1.0
- added link head_yaw_link, mass 1.0
- added link left_arch_tip, mass 1.0
- added link left_toe_tip, mass 1.0
Joints:
- added joint head_pitch: type continuous, parent head_yaw_link, child head_pitch_link, origin xyz=0 0 -0.1 rpy=0 0 0, axis 0 1 0
- added joint head_yaw: type continuous, parent trunk_link, child head_yaw_link, origin xyz=0 0 0.15 rpy=0 0 0, axis 0 0 1
- added joint left_arch: type fixed, parent left_ankle_roll_link, child left_arch_tip, origin xyz=0.02 0 -0.05 rpy=0 0 0
- added joint left_toe_tip_joint: type fixed, parent left_toe_link, child left_toe_tip, origin xyz=0.02 0 -0.04 rpy=0 0 0

Commit message: Adding bounding box to GrosBan foots

File: Data/GrosbanToe.urdf (robot description, URDF)
Before this commit: robot DummyRobot, 27 links, 26 joints
Links:
- added link right_arch_tip, mass 1.0
- added link right_toe_tip, mass 1.0
Joints:
- added joint right_arch: type fixed, parent right_ankle_roll_link, child right_arch_tip, origin xyz=0.04 -0.03 -0.06 rpy=0 0 0
- added joint right_toe_tip_joint: type fixed, parent right_toe_link, child right_toe_tip, origin xyz=0.02 -0.03 -0.06 rpy=0 0 0
- joint left_arch: origin xyz=0.02 0 -0.05 rpy=0 0 0 -> xyz=0.04 0.03 -0.06 rpy=0 0 0
- joint left_toe: origin xyz=0.1 0 0 rpy=0 0 0 -> xyz=0.15 0 0 rpy=0 0 0
- joint left_toe_tip_joint: origin xyz=0.02 0 -0.04 rpy=0 0 0 -> xyz=0.02 0.03 -0.06 rpy=0 0 0
- joint right_toe: origin xyz=0.1 0 0 rpy=0 0 0 -> xyz=0.15 0 0 rpy=0 0 0

Commit message: Importing manually CAD data for Grosban legs

File: Data/GrosbanToe.urdf (robot description, URDF)
Before this commit: robot DummyRobot, 29 links, 28 joints
Joints:
- joint left_ankle_pitch: origin xyz=0 0 -0.2 rpy=0 0 0 -> xyz=0 0 -0.25 rpy=0 0 0
- joint left_arch: origin xyz=0.04 0.03 -0.06 rpy=0 0 0 -> xyz=0.0216 0.015 -0.0667 rpy=0 0 0
- joint left_hip_yaw: origin xyz=0 0.1 -0.05 rpy=0 0 0 -> xyz=0 0.046375 0 rpy=0 0 0
- joint left_knee: origin xyz=0 0 -0.2 rpy=0 0 0 -> xyz=-0.014956 0 -0.249652 rpy=0 0 0
- joint left_shoulder_pitch: origin xyz=0 0.15 0.1 rpy=0 0 0 -> xyz=0 0.1 0.1 rpy=0 0 0
- joint left_toe: origin xyz=0.15 0 0 rpy=0 0 0 -> xyz=0.10132 0.015 -0.025 rpy=0 0 0
- joint left_toe_tip_joint: origin xyz=0.02 0.03 -0.06 rpy=0 0 0 -> xyz=0.021 0 -0.0417 rpy=0 0 0
- joint right_ankle_pitch: origin xyz=0 0 -0.2 rpy=0 0 0 -> xyz=0 0 -0.25 rpy=0 0 0
- joint right_arch: origin xyz=0.04 -0.03 -0.06 rpy=0 0 0 -> xyz=0.0216 -0.015 -0.0667 rpy=0 0 0
- joint right_hip_yaw: origin xyz=0 -0.1 -0.05 rpy=0 0 0 -> xyz=0 -0.046375 0 rpy=0 0 0
- joint right_knee: origin xyz=0 0 -0.2 rpy=0 0 0 -> xyz=-0.014956 0 -0.249652 rpy=0 0 0
- joint right_shoulder_pitch: origin xyz=0 -0.15 0.1 rpy=0 0 0 -> xyz=0 -0.1 0.1 rpy=0 0 0
- joint right_toe: origin xyz=0.15 0 0 rpy=0 0 0 -> xyz=0.10132 -0.015 -0.025 rpy=0 0 0
- joint right_toe_tip_joint: origin xyz=0.02 -0.03 -0.06 rpy=0 0 0 -> xyz=0.021 0 -0.0417 rpy=0 0 0

Commit message: Updating arms from grosban.urdf

File: Data/GrosbanToe.urdf (robot description, URDF)
Before this commit: robot DummyRobot, 29 links, 28 joints
Joints:
- joint head_yaw: origin xyz=0 0 0.15 rpy=0 0 0 -> xyz=0 0 0.21 rpy=0 0 0
- joint left_elbow: origin xyz=0 0 -0.1 rpy=0 0 0 -> xyz=0 0 -0.14 rpy=0 0 0
- joint left_hand: origin xyz=0 0 -0.1 rpy=0 0 0 -> xyz=0 0 -0.18 rpy=0 0 0
- joint left_shoulder_pitch: origin xyz=0 0.1 0.1 rpy=0 0 0 -> xyz=0 0.07 0.2 rpy=0 0 0
- joint right_elbow: origin xyz=0 0 -0.1 rpy=0 0 0 -> xyz=0 0 -0.14 rpy=0 0 0
- joint right_hand: origin xyz=0 0 -0.1 rpy=0 0 0 -> xyz=0 0 -0.18 rpy=0 0 0
- joint right_shoulder_pitch: origin xyz=0 -0.1 0.1 rpy=0 0 0 -> xyz=0 -0.07 0.2 rpy=0 0 0

Commit message: Updating size of Groban after femur reduction

File: Data/GrosbanToe.urdf (robot description, URDF)
Before this commit: robot DummyRobot, 29 links, 28 joints
Joints:
- joint left_knee: origin xyz=-0.014956 0 -0.249652 rpy=0 0 0 -> xyz=-0.014956 0 -0.179652 rpy=0 0 0
- joint right_knee: origin xyz=-0.014956 0 -0.249652 rpy=0 0 0 -> xyz=-0.014956 0 -0.179652 rpy=0 0 0
