Commit message: Mise à jour de Code et des modèles URDF pour utiliser la nouvelle convention de nomage moteurs

File: Data/grosban.urdf (robot description, URDF)
Before this commit: robot URDF, 26 links, 25 joints
Links:
- removed link left_arm_pitch_link
- removed link left_arm_roll_link
- removed link left_foot_pitch_link
- removed link left_foot_roll_link
- removed link pan_link
- removed link right_arm_pitch_link
- removed link right_arm_roll_link
- removed link right_foot_pitch_link
- removed link right_foot_roll_link
- removed link tilt_link
- added link head_pitch_link, mass 0.23099; collision mesh filename=package://URDF/meshes/tilt_link.STL; visual mesh filename=package://URDF/meshes/tilt_link.STL
- added link head_yaw_link, mass 0.0061892; collision mesh filename=package://URDF/meshes/pan_link.STL; visual mesh filename=package://URDF/meshes/pan_link.STL
- added link left_ankle_pitch_link, mass 0.34295; collision mesh filename=package://URDF/meshes/left_foot_pitch_link.STL; visual mesh filename=package://URDF/meshes/left_foot_pitch_link.STL
- added link left_ankle_roll_link, mass 0.35369; collision mesh filename=package://URDF/meshes/left_foot_roll_link.STL; visual mesh filename=package://URDF/meshes/left_foot_roll_link.STL
- added link left_shoulder_pitch_link, mass 0.021273; collision mesh filename=package://URDF/meshes/left_arm_pitch_link.STL; visual mesh filename=package://URDF/meshes/left_arm_pitch_link.STL
- added link left_shoulder_roll_link, mass 0.21057; collision mesh filename=package://URDF/meshes/left_arm_roll_link.STL; visual mesh filename=package://URDF/meshes/left_arm_roll_link.STL
- added link right_ankle_pitch_link, mass 0.34295; collision mesh filename=package://URDF/meshes/right_foot_pitch_link.STL; visual mesh filename=package://URDF/meshes/right_foot_pitch_link.STL
- added link right_ankle_roll_link, mass 0.35369; collision mesh filename=package://URDF/meshes/right_foot_roll_link.STL; visual mesh filename=package://URDF/meshes/right_foot_roll_link.STL
- added link right_shoulder_pitch_link, mass 0.021273; collision mesh filename=package://URDF/meshes/right_arm_pitch_link.STL; visual mesh filename=package://URDF/meshes/right_arm_pitch_link.STL
- added link right_shoulder_roll_link, mass 0.21057; collision mesh filename=package://URDF/meshes/right_arm_roll_link.STL; visual mesh filename=package://URDF/meshes/right_arm_roll_link.STL
Joints:
- removed joint left_arm_pitch
- removed joint left_arm_roll
- removed joint left_foot_pitch
- removed joint left_foot_roll
- removed joint pan
- removed joint right_arm_pitch
- removed joint right_arm_roll
- removed joint right_foot_pitch
- removed joint right_foot_roll
- removed joint tilt
- added joint head_pitch: type continuous, parent head_yaw_link, child head_pitch_link, origin xyz=0 0 0.0275 rpy=2.1684E-19 4.2352E-22 -0.00070549, axis 0 1 0
- added joint head_yaw: type continuous, parent trunk_link, child head_yaw_link, origin xyz=0.02642 0.0003237 0.21325 rpy=-0.001509 -5.6246E-07 0.00070549, axis 0 0 1
- added joint left_ankle_pitch: type continuous, parent left_knee_link, child left_ankle_pitch_link, origin xyz=0 0 -0.25 rpy=0 -2.6417E-16 0.0010782, axis 0 1 0
- added joint left_ankle_roll: type continuous, parent left_ankle_pitch_link, child left_ankle_roll_link, origin xyz=0 0 0 rpy=0 2.4074E-35 0, axis 1 0 0
- added joint left_shoulder_pitch: type continuous, parent trunk_link, child left_shoulder_pitch_link, origin xyz=0.010627 0.071185 0.20514 rpy=-3.4455E-19 3.1955E-16 -9.0974E-35, axis 0 1 0
- added joint left_shoulder_roll: type continuous, parent left_shoulder_pitch_link, child left_shoulder_roll_link, origin xyz=0 0.0325 -4.9044E-05 rpy=-0.001509 -5.6246E-07 0.00070549, axis 1 0 0
- added joint right_ankle_pitch: type continuous, parent right_knee_link, child right_ankle_pitch_link, origin xyz=0 0 -0.25 rpy=0 2.0615E-14 0.0010782, axis 0 1 0
- added joint right_ankle_roll: type continuous, parent right_ankle_pitch_link, child right_ankle_roll_link, origin xyz=0 0 0 rpy=-2.4652E-32 0 2.5178E-30, axis 1 0 0
- added joint right_shoulder_pitch: type continuous, parent trunk_link, child right_shoulder_pitch_link, origin xyz=0.010727 -0.070561 0.20536 rpy=0 0 0, axis 0 1 0
- added joint right_shoulder_roll: type continuous, parent right_shoulder_pitch_link, child right_shoulder_roll_link, origin xyz=0 -0.0325 4.9044E-05 rpy=-0.001509 -5.6246E-07 0.00070549, axis 1 0 0
- joint camera: parent tilt_link -> head_pitch_link
- joint left_elbow: parent left_arm_roll_link -> left_shoulder_roll_link
- joint left_foot_tip: parent left_foot_roll_link -> left_ankle_roll_link
- joint right_elbow: parent right_arm_roll_link -> right_shoulder_roll_link
- joint right_foot_tip: parent right_foot_roll_link -> right_ankle_roll_link

File: Data/sigmaban.urdf (robot description, URDF)
Before this commit: robot URDF, 26 links, 25 joints
Links:
- removed link left_arm_pitch_link
- removed link left_arm_roll_link
- removed link left_foot_pitch_link
- removed link left_foot_roll_link
- removed link pan_link
- removed link right_arm_pitch_link
- removed link right_arm_roll_link
- removed link right_foot_pitch_link
- removed link right_foot_roll_link
- removed link tilt_link
- added link head_pitch_link, mass 0.1509; collision mesh filename=package://URDF/meshes/tilt_link.STL; visual mesh filename=package://URDF/meshes/tilt_link.STL
- added link head_yaw_link, mass 0.010831; collision mesh filename=package://URDF/meshes/pan_link.STL; visual mesh filename=package://URDF/meshes/pan_link.STL
- added link left_ankle_pitch_link, mass 0.291968943886111; collision mesh filename=package://URDF/meshes/left_foot_pitch_link.STL; visual mesh filename=package://URDF/meshes/left_foot_pitch_link.STL
- added link left_ankle_roll_link, mass 0.076822; collision mesh filename=package://URDF/meshes/left_foot_roll_link.STL; visual mesh filename=package://URDF/meshes/left_foot_roll_link.STL
- added link left_shoulder_pitch_link, mass 0.0108311828445786; collision mesh filename=package://URDF/meshes/left_arm_pitch_link.STL; visual mesh filename=package://URDF/meshes/left_arm_pitch_link.STL
- added link left_shoulder_roll_link, mass 0.112091465246663; collision mesh filename=package://URDF/meshes/left_arm_roll_link.STL; visual mesh filename=package://URDF/meshes/left_arm_roll_link.STL
- added link right_ankle_pitch_link, mass 0.291968943886111; collision mesh filename=package://URDF/meshes/right_foot_pitch_link.STL; visual mesh filename=package://URDF/meshes/right_foot_pitch_link.STL
- added link right_ankle_roll_link, mass 0.0768216494717704; collision mesh filename=package://URDF/meshes/right_foot_roll_link.STL; visual mesh filename=package://URDF/meshes/right_foot_roll_link.STL
- added link right_shoulder_pitch_link, mass 0.0108311828445787; collision mesh filename=package://URDF/meshes/right_arm_pitch_link.STL; visual mesh filename=package://URDF/meshes/right_arm_pitch_link.STL
- added link right_shoulder_roll_link, mass 0.11209; collision mesh filename=package://URDF/meshes/right_arm_roll_link.STL; visual mesh filename=package://URDF/meshes/right_arm_roll_link.STL
Joints:
- removed joint left_arm_pitch
- removed joint left_arm_roll
- removed joint left_foot_pitch
- removed joint left_foot_rool
- removed joint pan
- removed joint right_arm_pitch
- removed joint right_arm_roll
- removed joint right_foot_pitch
- removed joint right_foot_roll
- removed joint tilt
- added joint head_pitch: type continuous, parent head_yaw_link, child head_pitch_link, origin xyz=0 0 0.046 rpy=1.3514E-14 9.7219E-31 -0.0010782, axis 0 1 0
- added joint head_yaw: type continuous, parent trunk_link, child head_yaw_link, origin xyz=0.02687 -2.9396E-05 0.1525 rpy=-1.3173E-14 1.4204E-17 -2.1314E-14, axis 0 0 1
- added joint left_ankle_pitch: type continuous, parent left_knee_link, child left_ankle_pitch_link, origin xyz=0 0 -0.105 rpy=0 0 0, axis 0 1 0
- added joint left_ankle_roll: type continuous, parent left_ankle_pitch_link, child left_ankle_roll_link, origin xyz=0 0 0 rpy=0 0 0, axis 1 0 0
- added joint left_shoulder_pitch: type continuous, parent trunk_link, child left_shoulder_pitch_link, origin xyz=0.0111273159824835 0.0463607067979427 0.141000000000005 rpy=4.91888973129517E-16 6.34190653024847E-17 -0.00107822069516516, axis 0 1 0
- added joint left_shoulder_roll: type continuous, parent left_shoulder_pitch_link, child left_shoulder_roll_link, origin xyz=0 0.046 0 rpy=7.30574676925163E-05 -6.34190653024847E-17 7.52316386533968E-37, axis 1 0 0
- added joint right_ankle_pitch: type continuous, parent right_knee_link, child right_ankle_pitch_link, origin xyz=0 0 -0.105 rpy=0 0 -0.0010782, axis 0 1 0
- added joint right_ankle_roll: type continuous, parent right_ankle_pitch_link, child right_ankle_roll_link, origin xyz=0 0 0 rpy=0 0 0, axis 1 0 0
- added joint right_shoulder_pitch: type continuous, parent trunk_link, child right_shoulder_pitch_link, origin xyz=0.0111273159824815 -0.0463847022119884 0.141000000000006 rpy=4.91888973129517E-16 6.34190653024847E-17 -0.00107822069516516, axis 0 1 0
- added joint right_shoulder_roll: type continuous, parent right_shoulder_pitch_link, child right_shoulder_roll_link, origin xyz=0 -0.046 0 rpy=-1.3665338392116E-14 -7.87720585415642E-08 0.00107822069514385, axis 1 0 0
- joint camera_fixed: parent tilt_link -> head_pitch_link
- joint left_elbow: parent left_arm_roll_link -> left_shoulder_roll_link
- joint left_foot_tip_fixed: parent left_foot_roll_link -> left_ankle_roll_link
- joint right_elbow: parent right_arm_roll_link -> right_shoulder_roll_link
- joint right_foot_tip_fixed: parent right_foot_roll_link -> right_ankle_roll_link

Commit message: Removing 7 cm from grosBan femur

File: Data/grosban.urdf (robot description, URDF)
Before this commit: robot URDF, 26 links, 25 joints
Joints:
- joint left_knee: origin xyz=-0.014956 -1.6126E-05 -0.24965 rpy=0 0 0 -> xyz=-0.014956 -1.6126E-05 -0.17965 rpy=0 0 0
- joint right_knee: origin xyz=-0.014956 -1.6126E-05 -0.24965 rpy=0 0 0 -> xyz=-0.014956 -1.6126E-05 -0.17965 rpy=0 0 0
