Commit message: Nouveau modèle dynamique de sigmaban 2016 avec la bonnes côtes et masses

File: Data/sigmaban_metabot.urdf (robot description, URDF)
Before this commit: robot metabot, 26 links, 25 joints
Links:
- link head_pitch: mass 0.078672 -> 0.081452; geometry collision box size=0.0354 0.0504 0.0353; visual mesh filename=package://urdf/2315e68be0ea2e6e80f047b6547c6a9dfbdc80f4.stl
- link head_yaw: mass 0.020112 -> 0.028492
- link left_ankle_pitch: mass 0.27798 -> 0.288805
- link left_ankle_roll: mass 0.138876 -> 0.196741
- link left_elbow: mass 0.117876 -> 0.136991
- link left_hip_pitch: mass 0.175404 -> 0.195989
- link left_hip_roll: mass 0.27798 -> 0.288805
- link left_hip_yaw: mass 0.022812 -> 0.032317
- link left_knee: mass 0.04344 -> 0.06154
- link left_shoulder_pitch: mass 0.020472 -> 0.029002
- link left_shoulder_roll: mass 0.127272 -> 0.150302
- link right_ankle_pitch: mass 0.27798 -> 0.288805
- link right_ankle_roll: mass 0.138876 -> 0.196741
- link right_elbow: mass 0.117876 -> 0.136991
- link right_hip_pitch: mass 0.175404 -> 0.195989
- link right_hip_roll: mass 0.27798 -> 0.288805
- link right_hip_yaw: mass 0.022812 -> 0.032317
- link right_knee: mass 0.04344 -> 0.06154
- link right_shoulder_pitch: mass 0.020472 -> 0.029002
- link right_shoulder_roll: mass 0.127272 -> 0.150302
- link trunk: mass 1.10899 -> 1.37255; geometry collision box size=0.0354 0.0504 0.0353; collision box size=0.0354 0.0504 0.0353
Joints:
- joint camera: origin xyz=-3.00754e-33 1.35447e-17 0.061 rpy=0 -0 0 -> xyz=0.01 1.59872e-17 0.062 rpy=0 -0 0
- joint head_yaw: origin xyz=0 0 0.153 rpy=0 -0 0 -> xyz=0.018 0 0.16725 rpy=0 -0 0
- joint left_hip_yaw: origin xyz=-0.018 0.0465 0 rpy=0 -0 0 -> xyz=0 0.0465 0.0205 rpy=0 -0 0
- joint left_shoulder_pitch: origin xyz=-0.018 0.0465 0.153 rpy=0 -0 0 -> xyz=0 0.0465 0.1585 rpy=0 -0 0
- joint right_hip_yaw: origin xyz=-0.018 -0.0465 0 rpy=0 -0 0 -> xyz=0 -0.0465 0.0205 rpy=0 -0 0
- joint right_shoulder_pitch: origin xyz=-0.018 -0.0465 0.153 rpy=0 -0 0 -> xyz=0 -0.0465 0.1585 rpy=0 -0 0
