Commit message: Correction des problèmes numérique de ForwardSimulation et prise en compte des contraintes de contacts

File: Data/pendulum_triple.urdf (robot description, URDF)
Before this commit: robot URDF, 4 links, 3 joints
Links:
- removed link base_link
- added link base2_link, mass 1.17617061217883
Joints:
- joint roll1: parent base_link -> base2_link

Commit message: Mise à jour de pendulum_triple pour les tests

File: Data/pendulum_triple.urdf (robot description, URDF)
Before this commit: robot URDF, 4 links, 3 joints
Links:
- added link tip_link, mass 0
Joints:
- added joint tip: type fixed, parent roll3_link, child tip_link, origin xyz=0.0 0.0 0.1 rpy=0.0 0.0 0.0, axis 0 0 0
