Commit message: Nouveau pieds de Mowgly avec les crampons plus cours

File: Data/sigmaban_metabot_cleats.urdf (robot description, URDF)
Before this commit: robot metabot, 34 links, 33 joints
Joints:
- joint left_cleat_1: origin xyz=0.063 0.043 -0.061 rpy=0 0 0 -> xyz=0.063 0.043 -0.056 rpy=0 0 0
- joint left_cleat_2: origin xyz=0.063 -0.037 -0.061 rpy=0 0 0 -> xyz=0.063 -0.037 -0.056 rpy=0 0 0
- joint left_cleat_3: origin xyz=-0.063 -0.037 -0.061 rpy=0 0 0 -> xyz=-0.063 -0.037 -0.056 rpy=0 0 0
- joint left_cleat_4: origin xyz=-0.063 0.043 -0.061 rpy=0 0 0 -> xyz=-0.063 0.043 -0.056 rpy=0 0 0
- joint left_foot_tip: origin xyz=0 0 -0.061 rpy=0 0 0 -> xyz=0 0 -0.056 rpy=0 0 0
- joint right_cleat_1: origin xyz=0.063 0.037 -0.061 rpy=0 0 0 -> xyz=0.063 0.037 -0.056 rpy=0 0 0
- joint right_cleat_2: origin xyz=0.063 -0.043 -0.061 rpy=0 0 0 -> xyz=0.063 -0.043 -0.056 rpy=0 0 0
- joint right_cleat_3: origin xyz=-0.063 -0.043 -0.061 rpy=0 0 0 -> xyz=-0.063 -0.043 -0.056 rpy=0 0 0
- joint right_cleat_4: origin xyz=-0.063 0.037 -0.061 rpy=0 0 0 -> xyz=-0.063 0.037 -0.056 rpy=0 0 0
- joint right_foot_tip: origin xyz=0 0 -0.061 rpy=0 0 0 -> xyz=0 0 -0.056 rpy=0 0 0
